File: hardware/TM Expander.kicad_pcb (KiCad board)
At the start: 2 copper layers, 80.1 x 127.9 mm, 32 parts

Commit message: work on the schematic mostly
Parts:
- added REF**: BAS70-04, Package_TO_SOT_SMD:SOT-23, F.Cu at (191.8, 60.0)
- added REF**: 0805L010YR, Fuse:Fuse_0805_2012Metric, F.Cu at (198.9, 48.5)
Other:
- board text added: "TAXI!"
