File: hardware/TM Expander.kicad_sch (KiCad schematic)
At the start: 0 parts

Commit message: work on the schematic mostly
Parts:
- added C1, C12, C2, C3, C4, C7, C8, C9: 100n, symbol Device:C
- added C10, C11, C13: 1u, symbol Device:C
- added C14, C15, C16, C17: 4.7n, symbol Device:C
- added C5, C6: 10u, symbol Device:C
- added D1: BAS70-04, Package_TO_SOT_SMD:SOT-23, symbol Diode:BAS40-04
- added F1, F2: 0805L010YR, symbol Device:Polyfuse
- added J1, J2, J3, J4: AudioJack2_SwitchT, symbol Connector_Audio:AudioJack2_SwitchT
- added J10: Conn_4A, symbol Connector_Generic:Conn_01x04
- added J11: POWER, symbol Connector_Generic:Conn_02x05_Odd_Even
- added J5: Conn_1A, symbol Connector_Generic:Conn_01x04
- added J6: Conn_1B, symbol Connector_Generic:Conn_01x04
- added J7: Conn_2A, symbol Connector_Generic:Conn_01x04
- added J8: Conn_2B, symbol Connector_Generic:Conn_01x04
- added J9: Conn_3A, symbol Connector_Generic:Conn_01x04
- added R1, R11, R13, R2, R3, R4, R7, R9: 200K, symbol Device:R
- added R10, R12, R6, R8: 33K, symbol Device:R
- added R5: 470, symbol Device:R
- added RV1, RV2, RV3, RV4: B10K, symbol Device:R_Potentiometer
- added U1: LM4040C10IDBZR, Package_TO_SOT_SMD:SOT-23, symbol Reference_Voltage:LM4040DBZ-2.0
- added U2: MCP1703AT-5002E/DB, Package_TO_SOT_SMD:SOT-223-3_TabPin2, symbol Regulator_Linear:MCP1703Ax-120xxDB
- added U3: MCP6004, symbol Amplifier_Operational:MCP6004
Connections:
- new net: J5.1 (Pin_1), R1.1
- new net: J5.2 (Pin_2), R2.1
- new net: J5.3 (Pin_3), R3.1
- new net: J5.4 (Pin_4), R4.1
- new net: J4.T, R4.2
- new net: J1.T, R1.2
- new net: J2.T, R2.2
- new net: J3.T, R3.2
- new net +12V: F1.2, J11.1 (Pin_1), J11.2 (Pin_2)
- new net +3V3: RV1.1, RV2.1, RV3.1, RV4.1
- new net +5V: C11.1, C12.1, C13.1, U2.3 (VO), U3.4 (V+)
- new net -12V: F2.2, J11.10 (Pin_10), J11.9 (Pin_9)
- new net AFREF_-10: C9.2, R5.1, U1.2 (A)
- new net AREF_-10: R11.2, R13.2, R7.2, R9.2
- new net CV1: C14.1, R6.1, U3.1
- new net CV2: C16.1, C17.1, R10.1, R12.1, U3.14, U3.7
- new net CV3: C15.1, R8.1, U3.8
- new net F_POT1: C1.1, J7.1 (Pin_1), RV1.2
- new net F_POT2: C2.1, J7.2 (Pin_2), RV2.2
- new net F_POT3: C3.1, J7.3 (Pin_3), RV3.2
- new net F_POT4: C4.1, J7.4 (Pin_4), RV4.2
- new net GND: C1.2, C10.2, C11.2, C12.2, C13.2, C2.2, C3.2, C4.2, C5.2, C6.1, C7.2, C8.1, C9.1, D1.3, J1.S, J11.3 (Pin_3), J11.4 (Pin_4), J11.5 (Pin_5), J11.6 (Pin_6), J11.7 (Pin_7), J11.8 (Pin_8), J2.S, J3.S, J4.S, RV1.3, RV2.3, RV3.3, RV4.3, U1.1 (K), U2.2 (GND), U3.10 (+), U3.11 (V-), U3.12 (+), U3.3 (+), U3.5 (+)
- new net H_CV1: C14.2, J6.1 (Pin_1), R6.2, R7.1, U3.2 (-)
- new net H_CV2: C16.2, C17.2, J6.2 (Pin_2), R10.2, R11.1, R12.2, R13.1, U3.13 (-), U3.6 (-)
- new net H_CV3: C15.2, J6.3 (Pin_3), R8.2, R9.1, U3.9 (-)
- new net H_CV4: J6.4 (Pin_4)
- new net POT1: J8.1 (Pin_1)
- new net POT2: J8.2 (Pin_2)
- new net POT3: J8.3 (Pin_3)
- new net POT4: J8.4 (Pin_4)
- new net VCC: C10.1, C5.1, C7.1, D1.1, F1.1, U2.1 (VI)
- new net VEE: C6.2, C8.2, D1.2, F2.1, R5.2
Other:
- note added: "POWER"
- note added: "TOP BOARD"
